File: project.sch (KiCad schematic (older format))
At the start: 20 parts, among them J2 Conn_01x04, J3 Conn_01x04, J4 Conn_01x04, J8 Conn_01x06, J9 Conn_01x04, Q1 BC547, Q2 BC547, Q3 BC547, Q4 BC547, Q5 BC547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

Commit message: Diverse Anpassung, umstellug uf SMD
Parts:
- removed A1: Arduino_UNO_R3, Modules:Arduino_UNO_R3_WithMountingHoles, symbol modules:Arduino_UNO_R3
- removed J2, J3, J4: Conn_01x04, Connectors_Phoenix:PhoenixContact_MC-G_04x3.81mm_Angled, symbol Connector:Conn_01x04
- removed J8: Conn_01x06, Connectors_Phoenix:PhoenixContact_MSTBA-G_06x5.08mm_Angled, symbol Connector:Conn_01x06
- removed J9: Conn_01x04, Connectors_Phoenix:PhoenixContact_MSTBA-G_04x5.08mm_Angled, symbol Connector:Conn_01x04
- removed Q1, Q2, Q3, Q4, Q5, Q6, Q7: BC547, TO_SOT_Packages_THT:TO-92_Molded_Narrow, symbol Transistor:BC547
- removed R1, R2, R3, R4, R5, R6, R7: 10k, Resistors_SMD:R_0805_HandSoldering, symbol device:R
- added A1: Arduino_Nano_v3.x, Modules:Arduino_Nano_WithMountingHoles, symbol MCU_Module:Arduino_Nano_v3.x
- added C1: 1uF, Capacitors_SMD:CP_Elec_8x10, symbol Device:C
- added J1, J2, J3, J4, J6: Conn_01x04, Connectors_Phoenix:PhoenixContact_MC-G_04x3.50mm_Angled, symbol Connector_Generic:Conn_01x04
- added J5: Conn_01x06, Connectors_Phoenix:PhoenixContact_MC-G_06x3.50mm_Angled, symbol Connector_Generic:Conn_01x06
- added Q1, Q2, Q3, Q4, Q5, Q6, Q7: BC848, TO_SOT_Packages_SMD:SOT-23_Handsoldering, symbol Transistor_BJT:BC848
- added R1, R2, R3, R4, R5, R6, R7: 10k, Resistors_SMD:R_1206_HandSoldering, symbol Device:R
- added R8: 47k, Resistors_SMD:R_1206_HandSoldering, symbol Device:R
Connections:
- net labels added: GND_NP, GND_Se, PWR_NP, PWR_Se, SIG_NP, Stell_DZ, Stell_GND
- net labels removed: 24V+, 24V-, Cutter
- wire segments 107 -> 114
Other:
- note added: "Drehzahlvorgabe"

Commit message: Fertiggestelltes Layout
Parts:
- added D1: LED, Diode_SMD:D_0805_2012Metric_Pad0.97x1.50mm_HandSolder, symbol Device:LED
- added J7: Conn_01x04, Connector_PinHeader_2.54mm:PinHeader_2x04_P2.54mm_Vertical, symbol Connector_Generic:Conn_01x08
- added J9: Conn_02x20_Odd_Even, symbol Connector_Generic:Conn_02x20_Odd_Even
- added Q8, Q9: BSS138, Package_TO_SOT_SMD:SOT-23, symbol Transistor_FET:BSS138
- added R10, R11, R12, R9: 10k, Resistor_SMD:R_0603_1608Metric_Pad0.84x1.00mm_HandSolder, symbol Device:R
- added R13: 220, Diode_SMD:D_0603_1608Metric_Pad0.67x1.00mm_HandSolder, symbol Device:R
Connections:
- net labels added: +3V3, GND, ID_SC, ID_SD, RXD, RX_5V, TXD, TX_5V
- wire segments 114 -> 150
- no-connect marks 10 -> 8
Other:
- moved on the sheet: R8

Commit message: Update auf vorhandene Bauteile & Korrektur 3D Objekte
Parts:
- removed Q8, Q9: BSS138, Package_TO_SOT_SMD:SOT-23, symbol Transistor_FET:BSS138
- added Q8, Q9: 2N7002, Package_TO_SOT_SMD:SOT-23_Handsoldering, symbol Transistor_FET:2N7002
- A1: footprint Modules:Arduino_Nano_WithMountingHoles -> Module:Arduino_Nano_WithMountingHoles
- D1: footprint Diode_SMD:D_0805_2012Metric_Pad0.97x1.50mm_HandSolder -> Diode_SMD:D_0603_1608Metric_Pad0.67x1.00mm_HandSolder
- J1, J2, J3, J4, J6: footprint Connectors_Phoenix:PhoenixContact_MC-G_04x3.50mm_Angled -> Connector_Phoenix_MC:PhoenixContact_MC_1,5_4-G-3.5_1x04_P3.50mm_Horizontal
- J5: footprint Connectors_Phoenix:PhoenixContact_MC-G_06x3.50mm_Angled -> Connector_Phoenix_MC:PhoenixContact_MC_1,5_6-G-3.5_1x06_P3.50mm_Horizontal
- J9: footprint (none) -> grbl_skycnc_adapter:pi-gpio
- Q1, Q2, Q3, Q4, Q5, Q6, Q7: footprint TO_SOT_Packages_SMD:SOT-23_Handsoldering -> Package_TO_SOT_SMD:SOT-23_Handsoldering
- R1, R2, R4, R8: footprint Resistors_SMD:R_1206_HandSoldering -> Resistor_SMD:R_1206_3216Metric_Pad1.24x1.80mm_HandSolder
- R10, R11, R12, R9: footprint Resistor_SMD:R_0603_1608Metric_Pad0.84x1.00mm_HandSolder -> Resistor_SMD:R_0805_2012Metric_Pad1.15x1.50mm_HandSolder
- R13: footprint Diode_SMD:D_0603_1608Metric_Pad0.67x1.00mm_HandSolder -> Resistor_SMD:R_0603_1608Metric_Pad0.84x1.00mm_HandSolder
- R3, R5, R6, R7: footprint Resistors_SMD:R_1206_HandSoldering -> Resistor_SMD:R_0805_2012Metric_Pad1.15x1.50mm_HandSolder
Connections:
- net labels removed: GND
- wire segments 150 -> 151
