File: project.kicad_pcb (KiCad board)
At the start: 2 copper layers, 20 parts, among them J2 Conn_01x04, J3 Conn_01x04, J4 Conn_01x04, J8 Conn_01x06, J9 Conn_01x04, Q1 BC547, Q2 BC547, Q3 BC547, Q4 BC547, Q5 BC547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

Commit message: Some improvements
Routing:
- net Earth: track 0.00 -> 11.2 mm
- net StepZ: track 0.18 -> 10.3 mm, vias 0 -> 1
Changed lines of the file:
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@@
     (thickness 1.6)
     (drawings 0)
-    (tracks 125)
+    (tracks 137)
     (zones 0)
     (modules 20)
@@
   (segment (start 31.242 94.742) (end 34.036 91.948) (width 0.5) (layer F.Cu) (net 1))
   (segment (start 34.036 91.948) (end 34.036 89.535) (width 0.5) (layer F.Cu) (net 1) (status 20))
+  (segment (start 83.439 91.44) (end 88.138 91.44) (width 0.5) (layer B.Cu) (net 2))
+  (segment (start 82.55 90.551) (end 83.439 91.44) (width 0.5) (layer B.Cu) (net 2))
+  (segment (start 88.138 91.44) (end 89.027 90.551) (width 0.5) (layer B.Cu) (net 2))
+  (segment (start 82.55 89.535) (end 82.55 90.551) (width 0.5) (layer B.Cu) (net 2))
+  (segment (start 89.027 90.551) (end 89.027 89.535) (width 0.5) (layer B.Cu) (net 2))
+  (segment (start 89.526999 90.940001) (end 89.281 91.186) (width 0.5) (layer F.Cu) (net 2))
+  (segment (start 89.027 89.535) (end 89.526999 90.034999) (width 0.5) (layer F.Cu) (net 2))
+  (segment (start 89.526999 90.034999) (end 89.526999 90.940001) (width 0.5) (layer F.Cu) (net 2))
   (segment (start 35.306 88.265) (end 35.306 83.82) (width 0.5) (layer F.Cu) (net 3) (status 30))
   (segment (start 51.689 88.265) (end 51.689 83.82) (width 0.5) (layer F.Cu) (net 4) (status 30))
@@
   (segment (start 89.847967 74.717998) (end 88.303976 76.261989) (width 0.5) (layer F.Cu) (net 19))
   (segment (start 89.847967 70.820824) (end 89.847967 74.717998) (width 0.5) (layer F.Cu) (net 19))
+  (segment (start 74.803 79.121) (end 74.803 73.533) (width 0.5) (layer B.Cu) (net 20))
+  (segment (start 74.803 73.533) (end 76.581 71.755) (width 0.5) (layer B.Cu) (net 20))
+  (segment (start 74.803 79.121) (end 74.803 81.12) (width 0.5) (layer F.Cu) (net 20))
+  (via (at 74.803 79.121) (size 1.6) (drill 0.8) (layers F.Cu B.Cu) (net 20))
   (segment (start 76.708 71.628) (end 76.581 71.755) (width 0.5) (layer F.Cu) (net 20) (status 30))
   (segment (start 73.910978 66.805022) (end 87.812094 66.805022) (width 0.5) (layer F.Cu) (net 21))

Commit message: Diverse Anpassung, umstellug uf SMD
Parts:
- removed J8: Conn_01x06, Connectors_Phoenix:PhoenixContact_MSTBA-G_06x5.08mm_Angled
- removed J9: Conn_01x04, Connectors_Phoenix:PhoenixContact_MSTBA-G_04x5.08mm_Angled
- added C1: 1uF, Capacitors_SMD:CP_Elec_8x10, F.Cu at (117.2, 130.1)
- added J1: Conn_01x04, Connectors_Phoenix:PhoenixContact_MC-G_04x3.50mm_Angled, F.Cu at (16.5, 146.1)
- added J5: Conn_01x06, Connectors_Phoenix:PhoenixContact_MC-G_06x3.50mm_Angled, F.Cu at (87.3, 146.1)
- added J6: Conn_01x04, Connectors_Phoenix:PhoenixContact_MC-G_04x3.50mm_Angled, F.Cu at (111.8, 146.1)
- added R0: 0, Resistors_SMD:R_2010_HandSoldering, F.Cu at (78.2, 120.8)
- added R0: 0, Resistors_SMD:R_2010_HandSoldering, F.Cu at (44.2, 111.2)
- added R8: 47k, Resistors_SMD:R_1206_HandSoldering, F.Cu at (117.2, 118.6)
- added REF**: KiCAD Logo, Symbols:Symbol_KiCAD-Logo_CopperAndSilkScreenTop, F.Cu at (172.7, 45.7)
- added REF***: OSHW-Logo2_7.3x6mm_Copper, Symbols:OSHW-Logo2_7.3x6mm_Copper, F.Cu at (161.3, 45.7)
- A1: value Arduino_UNO_R3 -> Arduino_Nano_v3.x; footprint Modules:Arduino_UNO_R3_WithMountingHoles -> Modules:Arduino_Nano_WithMountingHoles
- J2, J3, J4: footprint Connectors_Phoenix:PhoenixContact_MC-G_04x3.81mm_Angled -> Connectors_Phoenix:PhoenixContact_MC-G_04x3.50mm_Angled
- Q1, Q2, Q3, Q4, Q5, Q6, Q7: value BC547 -> BC848; footprint TO_SOT_Packages_THT:TO-92_Molded_Narrow -> TO_SOT_Packages_SMD:SOT-23_Handsoldering
- R1, R2, R3, R4, R5, R6, R7: footprint Resistors_SMD:R_0805_HandSoldering -> Resistors_SMD:R_1206_HandSoldering
- moved A1 82.2 mm to (58.4, 105.4), turned to 90 degrees
- moved Q5 52.2 mm to (52.7, 137.4), turned to 270 degrees
- moved Q6 51.3 mm to (61.4, 137.4), turned to 270 degrees
- moved R5 51.1 mm to (53.4, 128.8)
- moved Q7 50.6 mm to (70.2, 137.4), turned to 270 degrees
- moved Q3 50.2 mm to (35.2, 137.4), turned to 270 degrees
- moved R6 50.2 mm to (62.1, 128.8)
- moved J2 49.8 mm to (34.3, 146.1)
- moved Q4 49.6 mm to (44.0, 137.4), turned to 270 degrees
- moved R7 49.2 mm to (71.1, 128.8)
- moved R3 49.0 mm to (35.9, 128.8)
- moved J3 48.9 mm to (52.1, 146.1)
- moved Q1 48.8 mm to (17.8, 137.4), turned to 270 degrees
- moved Q2 48.4 mm to (26.5, 137.4), turned to 270 degrees
- moved R4 48.3 mm to (44.6, 128.8)
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Connections:
- A1 pad 1: Net-(A1-Pad1) -> (no net)
- A1 pad 10: FeedHold -> DirZ
- A1 pad 11: CycleStart/Resume -> StepperEN
- A1 pad 12: CoolantEnable -> LimitX
- A1 pad 13: Net-(A1-Pad13) -> LimitY
- A1 pad 14: Probe -> SpindlePWM
- A1 pad 15: Net-(A1-Pad15) -> LimitZ
- A1 pad 16: Net-(A1-Pad16) -> (no net)
- A1 pad 17: StepX -> (no net)
- A1 pad 18: StepY -> (no net)
- A1 pad 19: StepZ -> (no net)
- A1 pad 2: Net-(A1-Pad2) -> (no net)
- A1 pad 20: DirX -> (no net)
- A1 pad 21: DirY -> (no net)
- A1 pad 22: DirZ -> (no net)
- A1 pad 23: StepperEN -> (no net)
- A1 pad 24: LimitX -> Probe
- A1 pad 25: LimitY -> (no net)
- A1 pad 26: SpindlePWM -> (no net)
- A1 pad 27: LimitZ -> +5V
- A1 pad 28: SpindleDir -> (no net)
- A1 pad 3: Net-(A1-Pad3) -> (no net)
- A1 pad 30: Net-(A1-Pad30) -> (no net)
- A1 pad 4: Net-(A1-Pad4) -> Earth
- A1 pad 5: +5V -> StepX
- A1 pad 6: Earth -> StepY
- A1 pad 7: Earth -> StepZ
- A1 pad 8: Net-(A1-Pad8) -> DirX
- A1 pad 9: Reset/Abort -> DirY
- J2 pad 2: StepXOut -> StepYOut
- J2 pad 3: DirXOut -> DirYOut
- J3 pad 2: StepYOut -> StepZOut
- J3 pad 3: DirYOut -> DirZOut
- J4 pad 1: +5V -> Earth
- J4 pad 2: StepZOut -> Earth
- J4 pad 3: DirZOut -> Probe
- J4 pad 4: StepperENOut -> (no net)
- Q1 pad 1: StepXOut -> Net-(Q1-Pad1)
- Q1 pad 2: Net-(Q1-Pad2) -> Earth
- Q1 pad 3: Earth -> StepXOut
- Q2 pad 1: DirXOut -> Net-(Q2-Pad1)
- Q2 pad 2: Net-(Q2-Pad2) -> Earth
- Q2 pad 3: Earth -> DirXOut
- Q3 pad 1: StepYOut -> Net-(Q3-Pad1)
- Q3 pad 2: Net-(Q3-Pad2) -> Earth
- Q3 pad 3: Earth -> StepYOut
- Q4 pad 1: DirYOut -> Net-(Q4-Pad1)
- Q4 pad 2: Net-(Q4-Pad2) -> Earth
- Q4 pad 3: Earth -> DirYOut
- Q5 pad 1: StepZOut -> Net-(Q5-Pad1)
- Q5 pad 2: Net-(Q5-Pad2) -> Earth
- Q5 pad 3: Earth -> StepZOut
- Q6 pad 1: DirZOut -> Net-(Q6-Pad1)
- Q6 pad 2: Net-(Q6-Pad2) -> Earth
- Q6 pad 3: Earth -> DirZOut
- Q7 pad 1: StepperENOut -> Net-(Q7-Pad1)
- Q7 pad 2: Net-(Q7-Pad2) -> Earth
- Q7 pad 3: Earth -> StepperENOut
- R1 pad 1: StepX -> Net-(Q1-Pad1)
- R1 pad 2: Net-(Q1-Pad2) -> StepX
- R2 pad 1: Net-(Q2-Pad2) -> Net-(Q2-Pad1)
- R3 pad 1: Net-(Q3-Pad2) -> Net-(Q3-Pad1)
- R4 pad 1: Net-(Q4-Pad2) -> Net-(Q4-Pad1)
- R5 pad 1: Net-(Q5-Pad2) -> Net-(Q5-Pad1)
- R6 pad 1: Net-(Q6-Pad2) -> Net-(Q6-Pad1)
- R7 pad 1: Net-(Q7-Pad2) -> Net-(Q7-Pad1)
Routing:
- net Probe: track 85.1 -> 14.0 mm
- net StepY: track 58.0 -> 14.3 mm
- net SpindlePWM: track 0.00 -> 37.7 mm
- net /24V+: track 34.8 -> 0.00 mm
- net /Stell_DZ: track 0.00 -> 28.7 mm
- net LimitZ: track 70.0 -> 43.4 mm
- net StepperENOut: track 84.4 -> 58.2 mm
- net LimitX: track 42.7 -> 63.4 mm
- net StepperEN: track 44.0 -> 26.7 mm
- net DirY: track 61.5 -> 44.5 mm
- net DirX: track 42.6 -> 59.6 mm
- net +5V: track 150.3 -> 134.7 mm
- net DirZ: track 43.2 -> 29.4 mm
- net Earth: track 11.2 -> 0.00 mm
- net StepZ: track 10.3 -> 0.00 mm, vias 1 -> 0
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- removed copper zone on F.Cu, net Earth

Commit message: Fertiggestelltes Layout
Parts:
- removed R0 (x2): 0, Resistors_SMD:R_2010_HandSoldering
- removed the REF** at (172.7, 45.7)
- removed REF***: OSHW-Logo2_7.3x6mm_Copper, Symbols:OSHW-Logo2_7.3x6mm_Copper
- added +3V3: +3V3, TestPoint:TestPoint_Pad_D1.0mm, F.Cu at (134.8, 60.8)
- added +3V3: TestPoint_Pad_D1.0mm, TestPoint:TestPoint_Pad_D1.0mm, F.Cu at (193.2, 64.0)
- added +3V3: TestPoint_Pad_D1.0mm, TestPoint:TestPoint_Pad_D1.0mm, F.Cu at (187.5, 66.0)
- added +5V: +5V, TestPoint:TestPoint_Pad_D1.0mm, F.Cu at (129.8, 61.0)
- added 0: 0, Resistor_SMD:R_1206_3216Metric_Pad1.24x1.80mm_HandSolder, F.Cu at (168.8, 74.7)
- added 0: 0, Resistor_SMD:R_1206_3216Metric_Pad1.24x1.80mm_HandSolder, F.Cu at (165.6, 74.7)
- added 0: 0, Resistor_SMD:R_1206_3216Metric_Pad1.24x1.80mm_HandSolder, F.Cu at (162.3, 74.7)
- added 0: 0, Resistor_SMD:R_1206_3216Metric_Pad1.24x1.80mm_HandSolder, F.Cu at (180.2, 74.6)
- added 0: 0, Resistor_SMD:R_1206_3216Metric_Pad1.24x1.80mm_HandSolder, F.Cu at (130.8, 79.1)
- added ?: , RPi_Hat:RPi_Hat_Mounting_Hole, F.Cu at (191.0, 59.5)
- added ?: , RPi_Hat:RPi_Hat_Mounting_Hole, F.Cu at (191.0, 108.5)
- added ?: , RPi_Hat:RPi_Hat_Mounting_Hole, F.Cu at (133.0, 108.5)
- added D1: LED, Diode_SMD:D_0805_2012Metric_Pad0.97x1.50mm_HandSolder, F.Cu at (129.8, 68.6)
- added G***: LOGO, grbl_skycnc_adapter:sf_logo, F.Cu at (159.8, 118.7)
- added J7: Conn_01x04, Connector_PinHeader_2.54mm:PinHeader_2x04_P2.54mm_Vertical, F.Cu at (184.2, 80.3)
- added J9: Conn_02x20_Odd_Even, RPi_Hat:Pin_Header_Straight_2x20, F.Cu at (162.0, 59.5)
- added Q8: BSS138, Package_TO_SOT_SMD:SOT-23, F.Cu at (184.2, 70.0)
- added Q9: BSS138, Package_TO_SOT_SMD:SOT-23, F.Cu at (190.8, 70.0)
- added R10: 10k, Resistor_SMD:R_0603_1608Metric_Pad0.84x1.00mm_HandSolder, F.Cu at (184.2, 66.0)
- added R11: 10k, Resistor_SMD:R_0603_1608Metric_Pad0.84x1.00mm_HandSolder, F.Cu at (190.8, 75.0)
- added R12: 10k, Resistor_SMD:R_0603_1608Metric_Pad0.84x1.00mm_HandSolder, F.Cu at (190.8, 66.0)
- added R13: 220, Diode_SMD:D_0603_1608Metric_Pad0.67x1.00mm_HandSolder, F.Cu at (129.8, 64.8)
- added R9: 10k, Resistor_SMD:R_0603_1608Metric_Pad0.84x1.00mm_HandSolder, F.Cu at (184.2, 75.0)
- added REF**: OSHW-Logo_5.7x6mm_Copper, Symbol:OSHW-Logo_5.7x6mm_Copper, F.Cu at (164.2, 97.1)
- added Ref**: Val**, grbl_skycnc_adapter:sf_logo, F.Cu at (141.3, 94.5)
- R3, R5, R6, R7: footprint Resistors_SMD:R_1206_HandSoldering -> Resistor_SMD:R_0603_1608Metric_Pad0.84x1.00mm_HandSolder
- moved J1 121.8 mm to (104.4, 61.8), turned to 270 degrees
- moved R1 117.9 mm to (123.5, 75.2), turned to 0 degrees
- moved Q1 117.4 mm to (116.9, 74.5), turned to 180 degrees
- moved R2 108.3 mm to (123.5, 79.2), turned to 0 degrees
- moved Q2 107.4 mm to (116.9, 79.4), turned to 180 degrees
- moved R3 99.1 mm to (125.5, 86.5), turned to 0 degrees
- moved Q3 96.7 mm to (116.9, 85.6), turned to 180 degrees
- moved J2 96.6 mm to (104.4, 79.6), turned to 270 degrees
- moved R4 88.6 mm to (125.5, 92.7), turned to 0 degrees
- moved Q4 86.0 mm to (116.9, 91.8), turned to 180 degrees
- moved A1 81.4 mm to (136.5, 82.5)
- moved R5 77.2 mm to (124.5, 99.0), turned to 0 degrees
- moved Q7 75.7 mm to (136.5, 101.0)
- moved R7 75.6 mm to (140.8, 99.2), turned to 0 degrees
- moved Q5 75.3 mm to (116.9, 98.0), turned to 180 degrees
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Connections:
- A1 pad 1: (no net) -> TX_5V
- A1 pad 16: (no net) -> SpindleDir
- A1 pad 17: (no net) -> Net-(A1-Pad17)
- A1 pad 18: (no net) -> Net-(A1-Pad18)
- A1 pad 19: (no net) -> Reset/Abort
- A1 pad 2: (no net) -> RX_5V
- A1 pad 20: (no net) -> FeedHold
- A1 pad 21: (no net) -> CycleStart/Resume
- A1 pad 22: (no net) -> CoolantEnable
- A1 pad 23: (no net) -> Net-(A1-Pad23)
- A1 pad 25: (no net) -> Net-(A1-Pad25)
- A1 pad 26: (no net) -> Net-(A1-Pad26)
- A1 pad 28: (no net) -> Net-(A1-Pad28)
- A1 pad 3: (no net) -> Net-(A1-Pad3)
- A1 pad 30: (no net) -> Net-(A1-Pad30)
- J4 pad 4: (no net) -> /PWR_NP
- J5 pad 1: LimitZ -> LimitX
- J5 pad 3: LimitX -> LimitZ
- J6 pad 2: (no net) -> Net-(J6-Pad2)
- J6 pad 3: (no net) -> Net-(J6-Pad3)
Routing:
- net +5V: track 134.7 -> 232.3 mm, vias 0 -> 2
- net TX_5V: track 0.00 -> 95.8 mm
- net RX_5V: track 0.00 -> 91.5 mm
- net +3V3: track 0.00 -> 72.4 mm, vias 0 -> 2
- net RXD: track 0.00 -> 50.8 mm
- net Reset/Abort: track 0.00 -> 46.3 mm, vias 0 -> 2
- net CycleStart/Resume: track 0.00 -> 46.0 mm, vias 0 -> 2
- net TXD: track 0.00 -> 45.3 mm
- net StepZ: track 0.00 -> 38.4 mm
- net FeedHold: track 0.00 -> 35.8 mm, vias 0 -> 2
- net StepX: track 60.0 -> 27.7 mm, vias 0 -> 2
- net LimitX: track 63.4 -> 31.3 mm
- net DirX: track 59.6 -> 32.3 mm
- net Probe: track 14.0 -> 41.1 mm
- net LimitY: track 53.9 -> 29.9 mm
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- added copper zone on F.Cu, net Earth
Other:
- board outline added: 98.5 x 56 mm
- net class GND added: clearance 0.2, trace_width 0.25, via_dia 0.8, via_drill 0.4
- net class komm added: clearance 0.2, trace_width 0.25, via_dia 0.8, via_drill 0.4

Commit message: Update auf vorhandene Bauteile & Korrektur 3D Objekte
Parts:
- A1: footprint Modules:Arduino_Nano_WithMountingHoles -> Module:Arduino_Nano_WithMountingHoles
- D1: footprint Diode_SMD:D_0805_2012Metric_Pad0.97x1.50mm_HandSolder -> Diode_SMD:D_0603_1608Metric_Pad0.67x1.00mm_HandSolder
- J1, J2, J3, J4, J6: footprint Connectors_Phoenix:PhoenixContact_MC-G_04x3.50mm_Angled -> Connector_Phoenix_MC:PhoenixContact_MC_1,5_4-G-3.5_1x04_P3.50mm_Horizontal
- J5: footprint Connectors_Phoenix:PhoenixContact_MC-G_06x3.50mm_Angled -> Connector_Phoenix_MC:PhoenixContact_MC_1,5_6-G-3.5_1x06_P3.50mm_Horizontal
- J9: footprint RPi_Hat:Pin_Header_Straight_2x20 -> grbl_skycnc_adapter:pi-gpio; moved to B.Cu
- Q1, Q2, Q3, Q4, Q5, Q6, Q7: footprint TO_SOT_Packages_SMD:SOT-23_Handsoldering -> Package_TO_SOT_SMD:SOT-23_Handsoldering
- Q8, Q9: value BSS138 -> 2N7002; footprint Package_TO_SOT_SMD:SOT-23 -> Package_TO_SOT_SMD:SOT-23_Handsoldering
- R1, R2, R4, R8: footprint Resistors_SMD:R_1206_HandSoldering -> Resistor_SMD:R_1206_3216Metric_Pad1.24x1.80mm_HandSolder
- R10, R11, R12, R3, R5, R6, R7, R9: footprint Resistor_SMD:R_0603_1608Metric_Pad0.84x1.00mm_HandSolder -> Resistor_SMD:R_0805_2012Metric_Pad1.15x1.50mm_HandSolder
- R13: footprint Diode_SMD:D_0603_1608Metric_Pad0.67x1.00mm_HandSolder -> Resistor_SMD:R_0603_1608Metric_Pad0.84x1.00mm_HandSolder
- moved +3V3 2.11 mm to (191.2, 64.2)
- moved J4 1.77 mm to (122.7, 64.5)
- moved Ref** 0.50 mm to (141.3, 94.0)
- moved REF** 0.30 mm to (163.9, 97.1)
- moved J9 0.07 mm to (161.9, 59.5), turned to 270 degrees
Connections:
- J4 pad 4: /PWR_NP -> +5V
- J9 pad 6: GND -> Earth
Routing:
- net Probe: track 41.1 -> 44.3 mm
- net +5V: track 232.3 -> 235.3 mm
- net +3V3: track 72.4 -> 69.6 mm
- net StepperEN: track 28.5 -> 29.9 mm
- net TXD: track 45.3 -> 46.5 mm
- net LimitX: track 31.3 -> 32.5 mm
- net RXD: track 50.8 -> 49.9 mm
- net DirZ: track 48.5 -> 47.7 mm
- net LimitY: track 29.9 -> 30.5 mm

Commit message: Neuerzeugen der Plots zum Ätzen
Routing:
- net DirX: track 32.3 -> 31.2 mm
- net (no net): vias 0 -> 3
Changed lines of the file:
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@@
     (thickness 1.6)
     (drawings 7)
-    (tracks 311)
+    (tracks 312)
     (zones 0)
     (modules 48)
@@
     (visible_elements FFFFFF7F)
     (pcbplotparams
-      (layerselection 0x00020_7ffffffe)
+      (layerselection 0x00020_ffffffff)
       (usegerberextensions false)
       (usegerberattributes false)
@@
       (outputformat 4)
       (mirror false)
-      (drillshape 2)
+      (drillshape 1)
       (scaleselection 1)
       (outputdirectory ""))
@@
   (gr_line (start 194.5 59.5) (end 194.5 108.5) (layer Edge.Cuts) (width 0.15))
   (gr_line (start 96 56) (end 191 56) (layer Edge.Cuts) (width 0.15))
+  (via (at 133 108.499998) (size 2) (drill 0.4) (layers F.Cu B.Cu) (net 0))
+  (via (at 191 108.500002) (size 2) (drill 0.4) (layers F.Cu B.Cu) (net 0))
+  (via (at 191 59.5) (size 2) (drill 0.4) (layers F.Cu B.Cu) (net 0))
   (segment (start 113.155062 79.405062) (end 110.25 76.5) (width 0.5) (layer F.Cu) (net 1))
   (segment (start 115.385994 79.405062) (end 113.155062 79.405062) (width 0.5) (layer F.Cu) (net 1) (status 10))
@@
   (segment (start 129.25 77.5) (end 130.75 77.5) (width 0.5) (layer F.Cu) (net 10) (status 20))
   (segment (start 144.795 80.685) (end 146.66 82.55) (width 0.5) (layer F.Cu) (net 10) (status 20))
-  (segment (start 154.28 82.55) (end 154.28 81.41863) (width 0.5) (layer F.Cu) (net 11) (status 10))
-  (segment (start 154.28 81.41863) (end 152.11137 79.25) (width 0.5) (layer F.Cu) (net 11))
-  (segment (start 152.11137 79.25) (end 127 79.25) (width 0.5) (layer F.Cu) (net 11))
-  (segment (start 127 79.25) (end 125.5 79.25) (width 0.5) (layer F.Cu) (net 11) (status 20))
-  (segment (start 125.5 78.694008) (end 126.555992 79.75) (width 0.5) (layer F.Cu) (net 11) (status 10))
+  (segment (start 152.11137 79.25) (end 154.28 81.41863) (width 0.5) (layer F.Cu) (net 11))
+  (segment (start 125.0925 79.25) (end 152.11137 79.25) (width 0.5) (layer F.Cu) (net 11))
+  (segment (start 154.28 81.41863) (end 154.28 82.55) (width 0.5) (layer F.Cu) (net 11))
   (segment (start 148.05 86.55) (end 149.2 85.4) (width 0.5) (layer F.Cu) (net 12))
   (segment (start 149.2 85.4) (end 149.2 82.55) (width 0.5) (layer F.Cu) (net 12) (status 20))
   (segment (start 126.5 86.55) (end 148.05 86.55) (width 0.5) (layer F.Cu) (net 12) (status 10))
-  (segment (start 125.5 95.8) (end 125.5 91.75) (width 0.5) (layer F.Cu) (net 13))
+  (segment (start 125.5 91.5) (end 126.2 90.8) (width 0.5) (layer F.Cu) (net 13))
+  (segment (start 125.5 95.8) (end 125.5 91.5) (width 0.5) (layer F.Cu) (net 13))
+  (segment (start 126.2 90.8) (end 129.7 90.8) (width 0.5) (layer F.Cu) (net 13))
+  (segment (start 129.7 90.8) (end 132.87 87.63) (width 0.5) (layer F.Cu) (net 13))
+  (segment (start 132.87 87.63) (end 137.16 87.63) (width 0.5) (layer F.Cu) (net 13))
   (segment (start 125.5 96.696566) (end 125.5 95.8) (width 0.5) (layer F.Cu) (net 13))
   (segment (start 125.5 95.8) (end 125.5 96.2) (width 0.5) (layer F.Cu) (net 13))
   (segment (start 125.5 96.696566) (end 125.5 98.95) (width 0.5) (layer F.Cu) (net 13) (status 20))
   (segment (start 125.5 96.696566) (end 125.4625 96.734066) (width 0.5) (layer F.Cu) (net 13))
-  (segment (start 126.5 90.75) (end 129 90.75) (width 0.5) (layer F.Cu) (net 13))
-  (segment (start 129 90.75) (end 132.12 87.63) (width 0.5) (layer F.Cu) (net 13))
-  (segment (start 125.5 91.75) (end 126.5 90.75) (width 0.5) (layer F.Cu) (net 13))
-  (segment (start 132.12 87.63) (end 137.16 87.63) (width 0.5) (layer F.Cu) (net 13))
   (segment (start 151.74 84.26) (end 148.37 87.63) (width 0.5) (layer F.Cu) (net 13))
   (segment (start 148.37 87.63) (end 137.16 87.63) (width 0.5) (layer F.Cu) (net 13))

Commit message: Generated new Gerber files & new Kicad version
Connections:
- A1 pad 17: Net-(A1-Pad17) -> unconnected-(A1-3V3-Pad17)
- A1 pad 18: Net-(A1-Pad18) -> unconnected-(A1-AREF-Pad18)
- A1 pad 19: Reset/Abort -> Reset/Abort
- A1 pad 21: CycleStart/Resume -> CycleStart/Resume
- A1 pad 23: Net-(A1-Pad23) -> unconnected-(A1-A4-Pad23)
- A1 pad 25: Net-(A1-Pad25) -> unconnected-(A1-A6-Pad25)
- A1 pad 26: Net-(A1-Pad26) -> unconnected-(A1-A7-Pad26)
- A1 pad 28: Net-(A1-Pad28) -> unconnected-(A1-RESET-Pad28)
- A1 pad 3: Net-(A1-Pad3) -> unconnected-(A1-RESET-Pad3)
- A1 pad 30: Net-(A1-Pad30) -> unconnected-(A1-VIN-Pad30)
- J6 pad 2: Net-(J6-Pad2) -> unconnected-(J6-Pin_2-Pad2)
- J6 pad 3: Net-(J6-Pad3) -> unconnected-(J6-Pin_3-Pad3)
- J7 pad 4: CycleStart/Resume -> CycleStart/Resume
- J7 pad 5: Reset/Abort -> Reset/Abort
- J7 pad 6: Net-(J7-Pad6) -> unconnected-(J7-Pin_6-Pad6)
- J7 pad 7: Net-(J7-Pad7) -> unconnected-(J7-Pin_7-Pad7)
- J7 pad 8: Net-(J7-Pad8) -> unconnected-(J7-Pin_8-Pad8)
- J9 pad 11: Net-(J9-Pad11) -> unconnected-(J9-Pin_11-Pad11)
- J9 pad 12: Net-(J9-Pad12) -> unconnected-(J9-Pin_12-Pad12)
- J9 pad 13: Net-(J9-Pad13) -> unconnected-(J9-Pin_13-Pad13)
- J9 pad 14: Net-(J9-Pad14) -> unconnected-(J9-Pin_14-Pad14)
- J9 pad 15: Net-(J9-Pad15) -> unconnected-(J9-Pin_15-Pad15)
- J9 pad 16: Net-(J9-Pad16) -> unconnected-(J9-Pin_16-Pad16)
- J9 pad 17: Net-(J9-Pad17) -> unconnected-(J9-Pin_17-Pad17)
- J9 pad 18: Net-(J9-Pad18) -> unconnected-(J9-Pin_18-Pad18)
- J9 pad 19: Net-(J9-Pad19) -> unconnected-(J9-Pin_19-Pad19)
- J9 pad 20: Net-(J9-Pad20) -> unconnected-(J9-Pin_20-Pad20)
- J9 pad 21: Net-(J9-Pad21) -> unconnected-(J9-Pin_21-Pad21)
- J9 pad 22: Net-(J9-Pad22) -> unconnected-(J9-Pin_22-Pad22)
- J9 pad 23: Net-(J9-Pad23) -> unconnected-(J9-Pin_23-Pad23)
- J9 pad 24: Net-(J9-Pad24) -> unconnected-(J9-Pin_24-Pad24)
- J9 pad 25: Net-(J9-Pad25) -> unconnected-(J9-Pin_25-Pad25)
- J9 pad 26: Net-(J9-Pad26) -> unconnected-(J9-Pin_26-Pad26)
- J9 pad 29: Net-(J9-Pad29) -> unconnected-(J9-Pin_29-Pad29)
- J9 pad 3: Net-(J9-Pad3) -> unconnected-(J9-Pin_3-Pad3)
- J9 pad 30: Net-(J9-Pad30) -> unconnected-(J9-Pin_30-Pad30)
- J9 pad 31: Net-(J9-Pad31) -> unconnected-(J9-Pin_31-Pad31)
- J9 pad 32: Net-(J9-Pad32) -> unconnected-(J9-Pin_32-Pad32)
- J9 pad 33: Net-(J9-Pad33) -> unconnected-(J9-Pin_33-Pad33)
- J9 pad 34: Net-(J9-Pad34) -> unconnected-(J9-Pin_34-Pad34)
- J9 pad 35: Net-(J9-Pad35) -> unconnected-(J9-Pin_35-Pad35)
- J9 pad 36: Net-(J9-Pad36) -> unconnected-(J9-Pin_36-Pad36)
- J9 pad 37: Net-(J9-Pad37) -> unconnected-(J9-Pin_37-Pad37)
- J9 pad 38: Net-(J9-Pad38) -> unconnected-(J9-Pin_38-Pad38)
- J9 pad 39: Net-(J9-Pad39) -> unconnected-(J9-Pin_39-Pad39)
- J9 pad 40: Net-(J9-Pad40) -> unconnected-(J9-Pin_40-Pad40)
- J9 pad 5: Net-(J9-Pad5) -> unconnected-(J9-Pin_5-Pad5)
- J9 pad 7: Net-(J9-Pad7) -> unconnected-(J9-Pin_7-Pad7)
- J9 pad 9: Net-(J9-Pad9) -> unconnected-(J9-Pin_9-Pad9)
Routing:
- net DirY: track 33.9 -> 0.00 mm
- net +5V: track 235.3 -> 233.5 mm
- net TX_5V: track 95.8 -> 94.3 mm
- net Probe: track 44.3 -> 42.9 mm
- net DirZOut: track 11.9 -> 11.0 mm
- net DirZ: track 47.7 -> 47.2 mm
- net StepZ: track 38.9 -> 38.4 mm
- net (no net): vias 3 -> 0
Other:
- net class Default removed
- net class GND removed
- net class komm removed
